Commit message: Added imu and accurate noise values

File: urdf/mid360.xacro (robot description, xacro)
@@ -16,7 +16,11 @@
        xfer_format 0 = sensor_msgs/PointCloud2 (x y z intensity tag line timestamp)
                    1 = livox_ros_driver2/CustomMsg (as for FAST-LIO)
-     The built-in IMU (livox/imu) is not simulated. -->
+     The built-in IMU, also as the driver: sensor_msgs/Imu on ${imu_topic} at 200 Hz,
+     in ${name}_frame (axes aligned with it), acceleration in g. It sits at
+     ${name}_imu_link, (11.0, 23.29, -44.12) mm from the point cloud origin (manual),
+     so FAST-LIO's extrinsic_T is [-0.011, -0.02329, 0.04412], extrinsic_R identity.
+     Needs the world's gz-sim-imu-system. -->
 <robot xmlns:xacro="http://www.ros.org/wiki/xacro">
-  <xacro:macro name="mid360" params="parent *origin name:=livox topic:=livox/lidar xfer_format:=0">
+  <xacro:macro name="mid360" params="parent *origin name:=livox topic:=livox/lidar xfer_format:=0 imu_topic:=livox/imu">
     <joint name="${name}_base_joint" type="fixed">
       <parent link="${parent}"/>
@@ -87,4 +91,39 @@
           <frame_id>${name}_frame</frame_id>
           <xfer_format>${xfer_format}</xfer_format>
+          <!-- datasheet angular random error (1 sigma) -->
+          <angular_noise>0.15</angular_noise>
+        </plugin>
+      </sensor>
+    </gazebo>
+    <joint name="${name}_imu_joint" type="fixed">
+      <parent link="${name}_frame"/>
+      <child link="${name}_imu_link"/>
+      <origin xyz="0.011 0.02329 -0.04412"/>
+    </joint>
+    <link name="${name}_imu_link"/>
+    <gazebo reference="${name}_imu_link">
+      <sensor name="${name}_imu" type="imu">
+        <update_rate>200</update_rate>
+        <always_on>true</always_on>
+        <!-- gz only; the plugin publishes ${imu_topic} -->
+        <topic>${name}/imu_raw</topic>
+        <!-- white noise of the ICM-40609 (TDK datasheet DS-000330 v1.2, tables 1 and 2):
+             RMS noise at 100 Hz bandwidth (the Nyquist band of the 200 Hz output),
+             gyro 0.045 deg/s = 7.9e-4 rad/s, accel 1.00 mg = 9.8e-3 m/s^2. No bias. -->
+        <imu>
+          <angular_velocity>
+            <x><noise type="gaussian"><mean>0</mean><stddev>7.9e-4</stddev></noise></x>
+            <y><noise type="gaussian"><mean>0</mean><stddev>7.9e-4</stddev></noise></y>
+            <z><noise type="gaussian"><mean>0</mean><stddev>7.9e-4</stddev></noise></z>
+          </angular_velocity>
+          <linear_acceleration>
+            <x><noise type="gaussian"><mean>0</mean><stddev>9.8e-3</stddev></noise></x>
+            <y><noise type="gaussian"><mean>0</mean><stddev>9.8e-3</stddev></noise></y>
+            <z><noise type="gaussian"><mean>0</mean><stddev>9.8e-3</stddev></noise></z>
+          </linear_acceleration>
+        </imu>
+        <plugin filename="livox_gz_sim" name="livox_gz_sim::LivoxImu">
+          <topic>${imu_topic}</topic>
+          <frame_id>${name}_frame</frame_id>
         </plugin>
       </sensor>

Commit message: Added downsampling and intensity

File: urdf/mid360.xacro (robot description, xacro)
@@ -16,4 +16,6 @@
        xfer_format 0 = sensor_msgs/PointCloud2 (x y z intensity tag line timestamp)
                    1 = livox_ros_driver2/CustomMsg (as for FAST-LIO)
+     Reflectivity of a surface: <laser_retro> in its Gazebo visual, on Livox's scale (0-150
+     diffuse %, 151-255 retroreflective); 100 where unset.
      The built-in IMU, also as the driver: sensor_msgs/Imu on ${imu_topic} at 200 Hz,
      in ${name}_frame (axes aligned with it), acceleration in g. It sits at
@@ -22,5 +24,5 @@
      Needs the world's gz-sim-imu-system. -->
 <robot xmlns:xacro="http://www.ros.org/wiki/xacro">
-  <xacro:macro name="mid360" params="parent *origin name:=livox topic:=livox/lidar xfer_format:=0 imu_topic:=livox/imu">
+  <xacro:macro name="mid360" params="parent *origin name:=livox topic:=livox/lidar xfer_format:=0 imu_topic:=livox/imu downsample:=1">
     <joint name="${name}_base_joint" type="fixed">
       <parent link="${parent}"/>
@@ -93,4 +95,9 @@
           <!-- datasheet angular random error (1 sigma) -->
           <angular_noise>0.15</angular_noise>
+          <!-- every n-th pattern ray, to save CPU (n = 1: the real 200k points/s) -->
+          <downsample>${downsample}</downsample>
+          <!-- reflectivity (Livox 0-255) comes from the hit visual's <laser_retro>; this is for
+               surfaces without one -->
+          <default_reflectivity>100</default_reflectivity>
         </plugin>
       </sensor>

Commit message: Can take slices to better approximate real behavior

File: urdf/mid360.xacro (robot description, xacro)
@@ -13,5 +13,7 @@
      livox_gz_sim::LivoxLidar plugin samples it along Livox's recorded Mid-360
      pattern, 20k rays per 10 Hz frame, so coverage builds up over frames as on the
-     real sensor. It publishes as livox_ros_driver2 does, on ${topic} in ${name}_frame:
+     real sensor. slices:=n renders n images per frame and stamps each point with its
+     image's time (1: a snapshot, offsets 0; 5: offsets 0, 20, ..., 80 ms, motion skew as on
+     the real sensor, 5x the rendering). It publishes as livox_ros_driver2 does, on ${topic} in ${name}_frame:
        xfer_format 0 = sensor_msgs/PointCloud2 (x y z intensity tag line timestamp)
                    1 = livox_ros_driver2/CustomMsg (as for FAST-LIO)
@@ -24,5 +26,5 @@
      Needs the world's gz-sim-imu-system. -->
 <robot xmlns:xacro="http://www.ros.org/wiki/xacro">
-  <xacro:macro name="mid360" params="parent *origin name:=livox topic:=livox/lidar xfer_format:=0 imu_topic:=livox/imu downsample:=1">
+  <xacro:macro name="mid360" params="parent *origin name:=livox topic:=livox/lidar xfer_format:=0 imu_topic:=livox/imu downsample:=1 slices:=1">
     <joint name="${name}_base_joint" type="fixed">
       <parent link="${parent}"/>
@@ -53,5 +55,6 @@
     <gazebo reference="${name}_frame">
       <sensor name="${name}" type="gpu_lidar">
-        <update_rate>10</update_rate>
+        <!-- 10 Hz frames, each from ${slices} rendered image(s) -->
+        <update_rate>${10 * slices}</update_rate>
         <always_on>true</always_on>
         <visualize>false</visualize>
@@ -88,5 +91,8 @@
           <pattern>mid360.csv</pattern>
           <samples>20000</samples>
-          <point_rate>200000</point_rate>
+          <!-- 1: each frame is one snapshot, all point offsets 0 (Livox's ROS 1 plugin);
+               n: n images per frame, point offsets 0, 100/n, ... ms, so motion during a frame
+               skews the cloud as on the real sensor; n x the rendering cost -->
+          <slices>${slices}</slices>
           <line_count>4</line_count>
           <topic>${topic}</topic>

Commit message: Speeding up the interface

File: urdf/mid360.xacro (robot description, xacro)
@@ -10,10 +10,13 @@
      (the cable connector is on -X). FOV 360 deg x -7..52 deg, 0.1-40 m (10 %
      reflectivity), 200k points/s at 10 Hz.
-     Gazebo: a dense gpu_lidar (0.2 deg grid) renders a range image and the
+     Gazebo: a dense gpu_lidar (resolution:=0.2 deg grid) renders a range image and the
      livox_gz_sim::LivoxLidar plugin samples it along Livox's recorded Mid-360
      pattern, 20k rays per 10 Hz frame, so coverage builds up over frames as on the
      real sensor. slices:=n renders n images per frame and stamps each point with its
      image's time (1: a snapshot, offsets 0; 5: offsets 0, 20, ..., 80 ms, motion skew as on
-     the real sensor, 5x the rendering). It publishes as livox_ros_driver2 does, on ${topic} in ${name}_frame:
+     the real sensor, 5x the rendering). The rendering cost is about proportional to
+     slices / resolution^2; the angular error stays 0.15 deg up to a 0.5 deg grid (the
+     plugin adds less jitter on a coarser one). On an RTX 3050 laptop, with the scene alone:
+     slices 1 or 5 at 0.2, 10 at 0.3 or 0.4 run at real time. It publishes as livox_ros_driver2 does, on ${topic} in ${name}_frame:
        xfer_format 0 = sensor_msgs/PointCloud2 (x y z intensity tag line timestamp)
                    1 = livox_ros_driver2/CustomMsg (as for FAST-LIO)
@@ -26,5 +29,5 @@
      Needs the world's gz-sim-imu-system. -->
 <robot xmlns:xacro="http://www.ros.org/wiki/xacro">
-  <xacro:macro name="mid360" params="parent *origin name:=livox topic:=livox/lidar xfer_format:=0 imu_topic:=livox/imu downsample:=1 slices:=1">
+  <xacro:macro name="mid360" params="parent *origin name:=livox topic:=livox/lidar xfer_format:=0 imu_topic:=livox/imu downsample:=1 slices:=1 resolution:=0.2">
     <joint name="${name}_base_joint" type="fixed">
       <parent link="${parent}"/>
@@ -65,5 +68,5 @@
           <scan>
             <horizontal>
-              <samples>1801</samples>
+              <samples>${int(round(360 / resolution)) + 1}</samples>
               <min_angle>${-pi}</min_angle>
               <max_angle>${pi}</max_angle>
@@ -71,5 +74,5 @@
             <!-- covers the pattern's -7.2..52.2 deg -->
             <vertical>
-              <samples>300</samples>
+              <samples>${int(round(59.8 / resolution)) + 1}</samples>
               <min_angle>${radians(-7.4)}</min_angle>
               <max_angle>${radians(52.4)}</max_angle>
@@ -81,10 +84,5 @@
             <resolution>0.001</resolution>
           </range>
-          <!-- datasheet range precision 2 cm (1 sigma) at 10 m -->
-          <noise>
-            <type>gaussian</type>
-            <mean>0.0</mean>
-            <stddev>0.02</stddev>
-          </noise>
+          <!-- no <noise>: per pixel it is most of the sensor's cost; the plugin adds it -->
         </lidar>
         <plugin filename="livox_gz_sim" name="livox_gz_sim::LivoxLidar">
@@ -99,5 +97,7 @@
           <frame_id>${name}_frame</frame_id>
           <xfer_format>${xfer_format}</xfer_format>
-          <!-- datasheet angular random error (1 sigma) -->
+          <!-- datasheet range precision 2 cm (1 sigma) at 10 m, angular random error 0.15 deg
+               (1 sigma, including the dense image's pixel quantisation) -->
+          <range_noise>0.02</range_noise>
           <angular_noise>0.15</angular_noise>
           <!-- every n-th pattern ray, to save CPU (n = 1: the real 200k points/s) -->
