Commit message: Added mid360 scan pattern bases on actual hardware

File: urdf/demo.urdf.xacro (robot description, xacro)
@@ -2,4 +2,5 @@
 <!-- demo: a Mid-360 on top of a 1 m pole fixed to the world -->
 <robot name="mid360_demo" xmlns:xacro="http://www.ros.org/wiki/xacro">
+  <xacro:arg name="xfer_format" default="0"/>
   <xacro:include filename="$(find livox_gz_sim)/urdf/mid360.xacro"/>
   <link name="world"/>
@@ -23,5 +24,5 @@
     </inertial>
   </link>
-  <xacro:mid360 parent="pole">
+  <xacro:mid360 parent="pole" xfer_format="$(arg xfer_format)">
     <origin xyz="0 0 1.0"/>
   </xacro:mid360>

File: urdf/mid360.xacro (robot description, xacro)
@@ -1,9 +1,22 @@
 <?xml version="1.0"?>
-<!-- Livox Mid-360. Dimensions and the point cloud origin from the Mid-360 User
-     Manual (appendix drawing): 65 x 65 x 60 mm, 265 g, origin O 47 mm above the
-     bottom on the axis, +X on the logo side (the cable connector is on -X). -->
+<!-- Livox Mid-360 with its real (non-repetitive) scan pattern.
+       <xacro:include filename="$(find livox_gz_sim)/urdf/mid360.xacro"/>
+       <xacro:mid360 parent="base_link">
+         <origin xyz="..." rpy="..."/>
+       </xacro:mid360>
+     The origin places the centre of the sensor's bottom face. Dimensions and the
+     point cloud origin from the Mid-360 User Manual (appendix drawing): 65 x 65 x 60
+     mm, 265 g, origin O 47 mm above the bottom on the axis, +X on the logo side
+     (the cable connector is on -X). FOV 360 deg x -7..52 deg, 0.1-40 m (10 %
+     reflectivity), 200k points/s at 10 Hz.
+     Gazebo: a dense gpu_lidar (0.2 deg grid) renders a range image and the
+     livox_gz_sim::LivoxLidar plugin samples it along Livox's recorded Mid-360
+     pattern, 20k rays per 10 Hz frame, so coverage builds up over frames as on the
+     real sensor. It publishes as livox_ros_driver2 does, on ${topic} in ${name}_frame:
+       xfer_format 0 = sensor_msgs/PointCloud2 (x y z intensity tag line timestamp)
+                   1 = livox_ros_driver2/CustomMsg (as for FAST-LIO)
+     The built-in IMU (livox/imu) is not simulated. -->
 <robot xmlns:xacro="http://www.ros.org/wiki/xacro">
-  <xacro:macro name="mid360" params="parent *origin name:=livox topic:=livox/lidar">
-    <!-- origin: the centre of the sensor's bottom face -->
+  <xacro:macro name="mid360" params="parent *origin name:=livox topic:=livox/lidar xfer_format:=0">
     <joint name="${name}_base_joint" type="fixed">
       <parent link="${parent}"/>
@@ -32,25 +45,24 @@
     </joint>
     <link name="${name}_frame"/>
-    <!-- a plain grid lidar over the Mid-360's field of view for now:
-         360 deg x -7..52 deg, 0.1-40 m, 10 Hz, ~20k points per frame
-         (the real sensor gives 200k points/s) -->
     <gazebo reference="${name}_frame">
       <sensor name="${name}" type="gpu_lidar">
-        <topic>${topic}</topic>
-        <gz_frame_id>${name}_frame</gz_frame_id>
         <update_rate>10</update_rate>
         <always_on>true</always_on>
         <visualize>false</visualize>
+        <!-- the dense image, gz only; the plugin publishes ${topic} -->
+        <topic>${name}/dense_scan</topic>
+        <gz_frame_id>${name}_frame</gz_frame_id>
         <lidar>
           <scan>
             <horizontal>
-              <samples>360</samples>
-              <min_angle>-3.14159</min_angle>
-              <max_angle>3.14159</max_angle>
+              <samples>1801</samples>
+              <min_angle>${-pi}</min_angle>
+              <max_angle>${pi}</max_angle>
             </horizontal>
+            <!-- covers the pattern's -7.2..52.2 deg -->
             <vertical>
-              <samples>60</samples>
-              <min_angle>-0.12217</min_angle>
-              <max_angle>0.90757</max_angle>
+              <samples>300</samples>
+              <min_angle>${radians(-7.4)}</min_angle>
+              <max_angle>${radians(52.4)}</max_angle>
             </vertical>
           </scan>
@@ -58,12 +70,22 @@
             <min>0.1</min>
             <max>40.0</max>
-            <resolution>0.002</resolution>
+            <resolution>0.001</resolution>
           </range>
+          <!-- datasheet range precision 2 cm (1 sigma) at 10 m -->
           <noise>
             <type>gaussian</type>
-            <mean>0</mean>
-            <stddev>0.01</stddev>
+            <mean>0.0</mean>
+            <stddev>0.02</stddev>
           </noise>
         </lidar>
+        <plugin filename="livox_gz_sim" name="livox_gz_sim::LivoxLidar">
+          <pattern>mid360.csv</pattern>
+          <samples>20000</samples>
+          <point_rate>200000</point_rate>
+          <line_count>4</line_count>
+          <topic>${topic}</topic>
+          <frame_id>${name}_frame</frame_id>
+          <xfer_format>${xfer_format}</xfer_format>
+        </plugin>
       </sensor>
     </gazebo>

Commit message: add color in gazebo

File: urdf/demo.urdf.xacro (robot description, xacro)
@@ -13,4 +13,5 @@
       <origin xyz="0 0 0.5"/>
       <geometry><cylinder radius="0.02" length="1.0"/></geometry>
+      <material name="pole_grey"><color rgba="0.6 0.6 0.62 1"/></material>
     </visual>
     <collision>

Commit message: Added hap lidar as well.

File: urdf/demo.urdf.xacro (robot description, xacro)
@@ -1,5 +1,6 @@
 <?xml version="1.0"?>
-<!-- demo: a Mid-360 on top of a 1 m pole fixed to the world -->
-<robot name="mid360_demo" xmlns:xacro="http://www.ros.org/wiki/xacro">
+<!-- demo: a Livox lidar (model:=mid360 or hap) on top of a 1 m pole fixed to the world -->
+<robot name="livox_demo" xmlns:xacro="http://www.ros.org/wiki/xacro">
+  <xacro:arg name="model" default="mid360"/>
   <xacro:arg name="xfer_format" default="0"/>
   <xacro:arg name="slices" default="1"/>
@@ -7,4 +8,5 @@
   <xacro:arg name="downsample" default="1"/>
   <xacro:include filename="$(find livox_gz_sim)/urdf/mid360.xacro"/>
+  <xacro:include filename="$(find livox_gz_sim)/urdf/hap.xacro"/>
   <link name="world"/>
   <joint name="pole_joint" type="fixed">
@@ -28,7 +30,16 @@
     </inertial>
   </link>
-  <xacro:mid360 parent="pole" xfer_format="$(arg xfer_format)" slices="$(arg slices)"
-                resolution="$(arg resolution)" downsample="$(arg downsample)">
-    <origin xyz="0 0 1.0"/>
-  </xacro:mid360>
+  <xacro:if value="${'$(arg model)' == 'mid360'}">
+    <xacro:mid360 parent="pole" xfer_format="$(arg xfer_format)" slices="$(arg slices)"
+                  resolution="$(arg resolution)" downsample="$(arg downsample)">
+      <origin xyz="0 0 1.0"/>
+    </xacro:mid360>
+  </xacro:if>
+  <!-- the HAP looks along +X, at the box and the far wall -->
+  <xacro:if value="${'$(arg model)' == 'hap'}">
+    <xacro:hap parent="pole" xfer_format="$(arg xfer_format)" slices="$(arg slices)"
+               resolution="$(arg resolution)" downsample="$(arg downsample)">
+      <origin xyz="0 0 1.0"/>
+    </xacro:hap>
+  </xacro:if>
 </robot>

File: urdf/mid360.xacro (robot description, xacro)
@@ -10,17 +10,9 @@
      (the cable connector is on -X). FOV 360 deg x -7..52 deg, 0.1-40 m (10 %
      reflectivity), 200k points/s at 10 Hz.
-     Gazebo: a dense gpu_lidar (resolution:=0.2 deg grid) renders a range image and the
-     livox_gz_sim::LivoxLidar plugin samples it along Livox's recorded Mid-360
-     pattern, 20k rays per 10 Hz frame, so coverage builds up over frames as on the
-     real sensor. slices:=n renders n images per frame and stamps each point with its
-     image's time (1: a snapshot, offsets 0; 5: offsets 0, 20, ..., 80 ms, motion skew as on
-     the real sensor, 5x the rendering). The rendering cost is about proportional to
-     slices / resolution^2; the angular error stays 0.15 deg up to a 0.5 deg grid (the
-     plugin adds less jitter on a coarser one). On an RTX 3050 laptop, with the scene alone:
-     slices 1 or 5 at 0.2, 10 at 0.3 or 0.4 run at real time. It publishes as livox_ros_driver2 does, on ${topic} in ${name}_frame:
-       xfer_format 0 = sensor_msgs/PointCloud2 (x y z intensity tag line timestamp)
-                   1 = livox_ros_driver2/CustomMsg (as for FAST-LIO)
-     Reflectivity of a surface: <laser_retro> in its Gazebo visual, on Livox's scale (0-150
-     diffuse %, 151-255 retroreflective); 100 where unset.
+     Gazebo: see livox_lidar.xacro (slices, resolution, downsample, xfer_format, reflectivity).
+     The dense image spans the pattern's -7.2..52.2 deg with margin; range noise 2 cm and
+     angular error 0.15 deg (1 sigma, datasheet), the latter kept up to resolution 0.5. On an
+     RTX 3050 laptop, with the scene alone, slices 1 or 5 at 0.2 and 10 at 0.3 or 0.4 run at
+     real time.
      The built-in IMU, also as the driver: sensor_msgs/Imu on ${imu_topic} at 200 Hz,
      in ${name}_frame (axes aligned with it), acceleration in g. It sits at
@@ -29,4 +21,5 @@
      Needs the world's gz-sim-imu-system. -->
 <robot xmlns:xacro="http://www.ros.org/wiki/xacro">
+  <xacro:include filename="$(find livox_gz_sim)/urdf/livox_lidar.xacro"/>
   <xacro:macro name="mid360" params="parent *origin name:=livox topic:=livox/lidar xfer_format:=0 imu_topic:=livox/imu downsample:=1 slices:=1 resolution:=0.2">
     <joint name="${name}_base_joint" type="fixed">
@@ -56,57 +49,9 @@
     </joint>
     <link name="${name}_frame"/>
-    <gazebo reference="${name}_frame">
-      <sensor name="${name}" type="gpu_lidar">
-        <!-- 10 Hz frames, each from ${slices} rendered image(s) -->
-        <update_rate>${10 * slices}</update_rate>
-        <always_on>true</always_on>
-        <visualize>false</visualize>
-        <!-- the dense image, gz only; the plugin publishes ${topic} -->
-        <topic>${name}/dense_scan</topic>
-        <gz_frame_id>${name}_frame</gz_frame_id>
-        <lidar>
-          <scan>
-            <horizontal>
-              <samples>${int(round(360 / resolution)) + 1}</samples>
-              <min_angle>${-pi}</min_angle>
-              <max_angle>${pi}</max_angle>
-            </horizontal>
-            <!-- covers the pattern's -7.2..52.2 deg -->
-            <vertical>
-              <samples>${int(round(59.8 / resolution)) + 1}</samples>
-              <min_angle>${radians(-7.4)}</min_angle>
-              <max_angle>${radians(52.4)}</max_angle>
-            </vertical>
-          </scan>
-          <range>
-            <min>0.1</min>
-            <max>40.0</max>
-            <resolution>0.001</resolution>
-          </range>
-          <!-- no <noise>: per pixel it is most of the sensor's cost; the plugin adds it -->
-        </lidar>
-        <plugin filename="livox_gz_sim" name="livox_gz_sim::LivoxLidar">
-          <pattern>mid360.csv</pattern>
-          <samples>20000</samples>
-          <!-- 1: each frame is one snapshot, all point offsets 0 (Livox's ROS 1 plugin);
-               n: n images per frame, point offsets 0, 100/n, ... ms, so motion during a frame
-               skews the cloud as on the real sensor; n x the rendering cost -->
-          <slices>${slices}</slices>
-          <line_count>4</line_count>
-          <topic>${topic}</topic>
-          <frame_id>${name}_frame</frame_id>
-          <xfer_format>${xfer_format}</xfer_format>
-          <!-- datasheet range precision 2 cm (1 sigma) at 10 m, angular random error 0.15 deg
-               (1 sigma, including the dense image's pixel quantisation) -->
-          <range_noise>0.02</range_noise>
-          <angular_noise>0.15</angular_noise>
-          <!-- every n-th pattern ray, to save CPU (n = 1: the real 200k points/s) -->
-          <downsample>${downsample}</downsample>
-          <!-- reflectivity (Livox 0-255) comes from the hit visual's <laser_retro>; this is for
-               surfaces without one -->
-          <default_reflectivity>100</default_reflectivity>
-        </plugin>
-      </sensor>
-    </gazebo>
+    <xacro:livox_lidar_sensor name="${name}" topic="${topic}" xfer_format="${xfer_format}"
+      slices="${slices}" resolution="${resolution}" downsample="${downsample}"
+      pattern="mid360.csv" samples="20000" line_count="4"
+      h_min="-180" h_max="180" v_min="-7.4" v_max="52.4"
+      range_min="0.1" range_max="40.0" range_noise="0.02" angular_noise="0.15"/>
     <joint name="${name}_imu_joint" type="fixed">
       <parent link="${name}_frame"/>

Commit message: added publish freq

File: urdf/demo.urdf.xacro (robot description, xacro)
@@ -4,4 +4,5 @@
   <xacro:arg name="model" default="mid360"/>
   <xacro:arg name="xfer_format" default="0"/>
+  <xacro:arg name="publish_freq" default="10.0"/>
   <xacro:arg name="slices" default="1"/>
   <xacro:arg name="resolution" default="0.2"/>
@@ -31,6 +32,6 @@
   </link>
   <xacro:if value="${'$(arg model)' == 'mid360'}">
-    <xacro:mid360 parent="pole" xfer_format="$(arg xfer_format)" slices="$(arg slices)"
-                  resolution="$(arg resolution)" downsample="$(arg downsample)">
+    <xacro:mid360 parent="pole" xfer_format="$(arg xfer_format)" publish_freq="$(arg publish_freq)"
+                  slices="$(arg slices)" resolution="$(arg resolution)" downsample="$(arg downsample)">
       <origin xyz="0 0 1.0"/>
     </xacro:mid360>
@@ -38,6 +39,6 @@
   <!-- the HAP looks along +X, at the box and the far wall -->
   <xacro:if value="${'$(arg model)' == 'hap'}">
-    <xacro:hap parent="pole" xfer_format="$(arg xfer_format)" slices="$(arg slices)"
-               resolution="$(arg resolution)" downsample="$(arg downsample)">
+    <xacro:hap parent="pole" xfer_format="$(arg xfer_format)" publish_freq="$(arg publish_freq)"
+               slices="$(arg slices)" resolution="$(arg resolution)" downsample="$(arg downsample)">
       <origin xyz="0 0 1.0"/>
     </xacro:hap>

File: urdf/hap.xacro (robot description, xacro)
@@ -11,5 +11,6 @@
      FOV 120 x 25 deg, 0.5 m blind zone, 150 m at 10 % reflectivity, 452k points/s at
      10 Hz (Livox HAP specs and user manual).
-     Gazebo: see livox_lidar.xacro (slices, resolution, downsample, xfer_format, reflectivity).
+     Gazebo: see livox_lidar.xacro (publish_freq, slices, resolution, downsample,
+     xfer_format, reflectivity).
      The dense image spans the pattern's +-60.25 x +-13.25 deg with margin (7x fewer
      pixels than the Mid-360's); range noise 2 cm (1 sigma at 20 m) and angular error 0.1
@@ -20,5 +21,5 @@
 <robot xmlns:xacro="http://www.ros.org/wiki/xacro">
   <xacro:include filename="$(find livox_gz_sim)/urdf/livox_lidar.xacro"/>
-  <xacro:macro name="hap" params="parent *origin name:=livox topic:=livox/lidar xfer_format:=0 downsample:=1 slices:=1 resolution:=0.2">
+  <xacro:macro name="hap" params="parent *origin name:=livox topic:=livox/lidar xfer_format:=0 publish_freq:=10.0 downsample:=1 slices:=1 resolution:=0.2">
     <joint name="${name}_base_joint" type="fixed">
       <parent link="${parent}"/>
@@ -48,6 +49,6 @@
     <link name="${name}_frame"/>
     <xacro:livox_lidar_sensor name="${name}" topic="${topic}" xfer_format="${xfer_format}"
-      slices="${slices}" resolution="${resolution}" downsample="${downsample}"
-      pattern="hap.csv" samples="45200" line_count="1"
+      publish_freq="${publish_freq}" slices="${slices}" resolution="${resolution}" downsample="${downsample}"
+      pattern="hap.csv" point_rate="452000" line_count="1"
       h_min="-60.4" h_max="60.4" v_min="-13.4" v_max="13.4"
       range_min="0.5" range_max="150.0" range_noise="0.02" angular_noise="0.1"/>

File: urdf/livox_lidar.xacro (robot description, xacro)
@@ -5,9 +5,10 @@
      elevation v_min..v_max, in deg) renders a range image and the
      livox_gz_sim::LivoxLidar plugin samples it along Livox's recorded scan pattern,
-     `samples` rays per 10 Hz frame, so coverage builds up over frames as on the real
-     sensor. slices:=n renders n images per frame and stamps each point with its image's
-     time (1: a snapshot, offsets 0; 5: offsets 0, 20, ..., 80 ms, motion skew as on the
-     real sensor, 5x the rendering). The rendering cost is about proportional to
-     slices x FOV / resolution^2; the angular error stays angular_noise as long as
+     point_rate / publish_freq rays per frame (the driver's publish_freq, Hz: a frame is
+     what one message carries), so coverage builds up over frames as on the real sensor.
+     slices:=n renders n images per frame and stamps each point with its image's time
+     (1: a snapshot, offsets 0; 5 at 10 Hz: offsets 0, 20, ..., 80 ms, motion skew as on
+     the real sensor, 5x the rendering). The rendering cost is about proportional to
+     slices x publish_freq x FOV / resolution^2; the angular error stays angular_noise as long as
      resolution / sqrt(12) < angular_noise (the plugin adds less jitter on a coarser grid).
      It publishes as livox_ros_driver2 does, on ${topic} in ${name}_frame:
@@ -18,10 +19,10 @@
 <robot xmlns:xacro="http://www.ros.org/wiki/xacro">
   <xacro:macro name="livox_lidar_sensor"
-               params="name topic xfer_format slices resolution downsample pattern samples line_count
+               params="name topic xfer_format publish_freq slices resolution downsample pattern point_rate line_count
                        h_min h_max v_min v_max range_min range_max range_noise angular_noise">
     <gazebo reference="${name}_frame">
       <sensor name="${name}" type="gpu_lidar">
-        <!-- 10 Hz frames, each from ${slices} rendered image(s) -->
-        <update_rate>${10 * slices}</update_rate>
+        <!-- ${publish_freq} Hz frames, each from ${slices} rendered image(s) -->
+        <update_rate>${publish_freq * slices}</update_rate>
         <always_on>true</always_on>
         <visualize>false</visualize>
@@ -51,7 +52,8 @@
         <plugin filename="livox_gz_sim" name="livox_gz_sim::LivoxLidar">
           <pattern>${pattern}</pattern>
-          <samples>${samples}</samples>
+          <!-- rays per frame -->
+          <samples>${int(round(point_rate / publish_freq))}</samples>
           <!-- 1: each frame is one snapshot, all point offsets 0 (Livox's ROS 1 plugin);
-               n: n images per frame, point offsets 0, 100/n, ... ms, so motion during a frame
+               n: n images per frame, point offsets 0, 1/n, ... of a frame, so motion during it
                skews the cloud as on the real sensor; n x the rendering cost -->
           <slices>${slices}</slices>

File: urdf/mid360.xacro (robot description, xacro)
@@ -10,5 +10,6 @@
      (the cable connector is on -X). FOV 360 deg x -7..52 deg, 0.1-40 m (10 %
      reflectivity), 200k points/s at 10 Hz.
-     Gazebo: see livox_lidar.xacro (slices, resolution, downsample, xfer_format, reflectivity).
+     Gazebo: see livox_lidar.xacro (publish_freq, slices, resolution, downsample,
+     xfer_format, reflectivity).
      The dense image spans the pattern's -7.2..52.2 deg with margin; range noise 2 cm and
      angular error 0.15 deg (1 sigma, datasheet), the latter kept up to resolution 0.5. On an
@@ -22,5 +23,5 @@
 <robot xmlns:xacro="http://www.ros.org/wiki/xacro">
   <xacro:include filename="$(find livox_gz_sim)/urdf/livox_lidar.xacro"/>
-  <xacro:macro name="mid360" params="parent *origin name:=livox topic:=livox/lidar xfer_format:=0 imu_topic:=livox/imu downsample:=1 slices:=1 resolution:=0.2">
+  <xacro:macro name="mid360" params="parent *origin name:=livox topic:=livox/lidar xfer_format:=0 publish_freq:=10.0 imu_topic:=livox/imu downsample:=1 slices:=1 resolution:=0.2">
     <joint name="${name}_base_joint" type="fixed">
       <parent link="${parent}"/>
@@ -50,6 +51,6 @@
     <link name="${name}_frame"/>
     <xacro:livox_lidar_sensor name="${name}" topic="${topic}" xfer_format="${xfer_format}"
-      slices="${slices}" resolution="${resolution}" downsample="${downsample}"
-      pattern="mid360.csv" samples="20000" line_count="4"
+      publish_freq="${publish_freq}" slices="${slices}" resolution="${resolution}" downsample="${downsample}"
+      pattern="mid360.csv" point_rate="200000" line_count="4"
       h_min="-180" h_max="180" v_min="-7.4" v_max="52.4"
       range_min="0.1" range_max="40.0" range_noise="0.02" angular_noise="0.15"/>
