Commit message: Setting defaults

File: urdf/demo.urdf.xacro (robot description, xacro)
@@ -5,6 +5,7 @@
   <xacro:arg name="xfer_format" default="0"/>
   <xacro:arg name="publish_freq" default="10.0"/>
-  <xacro:arg name="slices" default="1"/>
-  <xacro:arg name="resolution" default="0.2"/>
+  <xacro:arg name="slices" default="5"/>
+  <!-- empty: the model's default -->
+  <xacro:arg name="resolution" default=""/>
   <xacro:arg name="downsample" default="1"/>
   <xacro:include filename="$(find livox_gz_sim)/urdf/mid360.xacro"/>

File: urdf/hap.xacro (robot description, xacro)
@@ -16,4 +16,6 @@
      pixels than the Mid-360's); range noise 2 cm (1 sigma at 20 m) and angular error 0.1
      deg (1 sigma, datasheet "< 0.1"), the latter kept up to resolution 0.34.
+     Defaults slices 5, resolution 0.2 (empty: the same): 3.5x real time on an RTX 3050
+     laptop with the demo scene alone.
      Livox's recorded HAP pattern is 2.31 s long (it was cut at 2^20 rows), so it
      repeats every 23.2 frames where the real one does not. line = point index % 6, as
@@ -21,5 +23,6 @@
 <robot xmlns:xacro="http://www.ros.org/wiki/xacro">
   <xacro:include filename="$(find livox_gz_sim)/urdf/livox_lidar.xacro"/>
-  <xacro:macro name="hap" params="parent *origin name:=livox topic:=livox/lidar xfer_format:=0 publish_freq:=10.0 downsample:=1 slices:=1 resolution:=0.2">
+  <xacro:macro name="hap" params="parent *origin name:=livox topic:=livox/lidar xfer_format:=0 publish_freq:=10.0 downsample:=1 slices:=5 resolution:=0.2">
+    <xacro:property name="res" value="${float(resolution) if str(resolution).strip() else 0.2}"/>
     <joint name="${name}_base_joint" type="fixed">
       <parent link="${parent}"/>
@@ -49,5 +52,5 @@
     <link name="${name}_frame"/>
     <xacro:livox_lidar_sensor name="${name}" topic="${topic}" xfer_format="${xfer_format}"
-      publish_freq="${publish_freq}" slices="${slices}" resolution="${resolution}" downsample="${downsample}"
+      publish_freq="${publish_freq}" slices="${slices}" resolution="${res}" downsample="${downsample}"
       pattern="hap.csv" point_rate="452000" line_count="6"
       h_min="-60.4" h_max="60.4" v_min="-13.4" v_max="13.4"

File: urdf/mid360.xacro (robot description, xacro)
@@ -13,7 +13,7 @@
      xfer_format, reflectivity).
      The dense image spans the pattern's -7.2..52.2 deg with margin; range noise 2 cm and
-     angular error 0.15 deg (1 sigma, datasheet), the latter kept up to resolution 0.5. On an
-     RTX 3050 laptop, with the scene alone, slices 1 or 5 at 0.2 and 10 at 0.3 or 0.4 run at
-     real time.
+     angular error 0.15 deg (1 sigma, datasheet), the latter kept up to resolution 0.5.
+     Defaults slices 5 (points 0, 20, ..., 80 ms into a frame), resolution 0.4 (empty: the
+     same): 2.7x real time on an RTX 3050 laptop with the demo scene alone (0.2: 1.0x).
      The built-in IMU, also as the driver: sensor_msgs/Imu on ${imu_topic} at 200 Hz,
      in ${name}_frame (axes aligned with it), acceleration in g. It sits at
@@ -23,5 +23,6 @@
 <robot xmlns:xacro="http://www.ros.org/wiki/xacro">
   <xacro:include filename="$(find livox_gz_sim)/urdf/livox_lidar.xacro"/>
-  <xacro:macro name="mid360" params="parent *origin name:=livox topic:=livox/lidar xfer_format:=0 publish_freq:=10.0 imu_topic:=livox/imu downsample:=1 slices:=1 resolution:=0.2">
+  <xacro:macro name="mid360" params="parent *origin name:=livox topic:=livox/lidar xfer_format:=0 publish_freq:=10.0 imu_topic:=livox/imu downsample:=1 slices:=5 resolution:=0.4">
+    <xacro:property name="res" value="${float(resolution) if str(resolution).strip() else 0.4}"/>
     <joint name="${name}_base_joint" type="fixed">
       <parent link="${parent}"/>
@@ -51,5 +52,5 @@
     <link name="${name}_frame"/>
     <xacro:livox_lidar_sensor name="${name}" topic="${topic}" xfer_format="${xfer_format}"
-      publish_freq="${publish_freq}" slices="${slices}" resolution="${resolution}" downsample="${downsample}"
+      publish_freq="${publish_freq}" slices="${slices}" resolution="${res}" downsample="${downsample}"
       pattern="mid360.csv" point_rate="200000" line_count="4"
       h_min="-180" h_max="180" v_min="-7.4" v_max="52.4"
